File: hw/nrf_mcu.kicad_sch (KiCad schematic)
At the start: 6 parts

Commit message: nrf side system diagram
Parts:
- added C?: 0.5pF, symbol Device:C
- added C?: DNP, symbol Device:C
- added C?: 0.8pF, symbol Device:C
- added C?: NP0 +-1%, symbol Device:C
- added C?: C, symbol Device:C
- L?: value L -> 4.7nH
Connections:
- net at Y?.1: now also C?.1
- net GND: now reaches Y?.2
- net GND: now also J?.2 (Ext), Y?.4, C?.2, C?.2, C?.2, C?.2, C?.2
- net at Y?.3: now also C?.1
- net ANT: now reaches J?.1 (In)
- net at L?.1: now also C?.1
- net RF: now reaches L?.2
- net RF: now also C?.1, C?.1
Other:
- note added: "* USB IO? * SWD/JTAG? * NFC? * GPIO mappings? (Section 7) * Flash memory (QSPI)? * Ordering codes & Variations?"
- note added: "32 MHz Oscillator"
- note added: "32.768kHz Oscillator"
- note added: "Analog SW"
- note added: "Battery"
- note added: "Buttons"
- note added: "Current Measurement"
- note added: "Debug In"
- note added: "Debug Out"
- note added: "Ext. PSU"
- note added: "External QSPI Flash"
- note added: "GPIO"
- note added: "GPIO Flash memory pin Solder bridge for memory use (default: shorted) Solder bridge for GPIO use (default: open) 0.17 CS SB13 SB23 0.19 SCLK SB11 SB21 0.20 SIO_0/SI SB12 SB22 0.21 SIO_1/SO SB14 SB24 0.22 SIO_2/WP SB15 SB25 0.23 SIO_3/HOLD SB10 SB20"
- note added: "IF Boot/Reset"
- note added: "IF MCU USB"
- note added: "Interface MCU"
- note added: "LEDs"
- note added: "Li-Ion"
- note added: "Power Supply"
- note added: "Power Sw"
- note added: "RF Connector"
- note added: "RF Matching Network"
- note added: "The memory is connected to the chip using the following GPIOs:"
- note added: "The nRF52840 DK has a 64 Mb external flash memory. The memory is a multi-I/O memory supporting both regular SPI and Quad SPI."
- note added: "f 32.000MHz +/- 10ppm ESR 40${R} C_{L} 8pF D_{L} 100${mu}W"
- note added: "four-component RF match is recommended for new designs"
- note added: "nRF Power Source SW"
- note added: "nRF USB"
- note added: "nRF52840"
- moved on the sheet: J?, L?, Y?

Commit message: Xtal values
Parts:
- removed C?: C, symbol Device:C
- added C? (x2): 22.8pF, NP0, 1%, symbol Device:C
- C?: value NP0 +-1% -> 10pF, NP0, 0.1%
- C?: value C -> 10pF, NP0, 0.1%
Connections:
- net GND: now also Y?.2, Y?.4, C?.2, C?.2
- net at Y?.1: now also C?.1
- net at Y?.3: now also C?.1
Other:
- note added: "12.5 == 1.05 + (cL1*cL2)/(cL1 + cL2) --------------------------------------- Result: {12.44, {cL1 -> 22.79, cL2 -> 22.79}}"
- note added: "8 == 3 + (cL1*cL2)/(cL1 + cL2) --------------------------------------- Result: {7.996, {cL1 -> 9.99, cL2 -> 9.992}}"
- note removed: "f 32.000MHz +/- 10ppm ESR 40${R} C_{L} 8pF D_{L} 100${mu}W"
- moved on the sheet: Y?
Changed lines of the file:
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@@
   (junction (at 336.55 63.5) (diameter 0) (color 0 0 0 0)
   )
+  (junction (at -13.97 85.09) (diameter 0) (color 0 0 0 0)
+  )
   (polyline (pts (xy 100.33 -41.91) (xy 85.09 -41.91))
     (stroke (width 0) (type default) (color 0 0 0 0))
@@
     (stroke (width 0) (type default) (color 0 0 0 0))
   )
+  (wire (pts (xy -13.97 85.09) (xy -13.97 90.17))
+    (stroke (width 0) (type default) (color 0 0 0 0))
+  )
   (polyline (pts (xy 187.96 -58.42) (xy 208.28 -69.85))
     (stroke (width 0) (type default) (color 0 0 0 0))
   )
+  (wire (pts (xy -26.67 80.01) (xy -26.67 81.28))
+    (stroke (width 0) (type default) (color 0 0 0 0))
+  )
   (wire (pts (xy 210.82 55.88) (xy 201.93 55.88))
     (stroke (width 0) (type default) (color 0 0 0 0))
@@
     (stroke (width 0) (type default) (color 0 0 0 0))
   )
+  (wire (pts (xy -1.27 81.28) (xy -1.27 80.01))
+    (stroke (width 0) (type default) (color 0 0 0 0))
+  )
   (polyline (pts (xy 280.67 -64.77) (xy 283.21 -62.23))
     (stroke (width 0) (type default) (color 0 0 0 0))
@@
     (stroke (width 0) (type default) (color 0 0 0 0))
   )
+  (wire (pts (xy -17.78 80.01) (xy -26.67 80.01))
+    (stroke (width 0) (type default) (color 0 0 0 0))
+  )
   (polyline (pts (xy 243.84 -53.34) (xy 251.46 -53.34))
     (stroke (width 0) (type default) (color 0 0 0 0))
   )
+  (wire (pts (xy -10.16 80.01) (xy -1.27 80.01))
+    (stroke (width 0) (type default) (color 0 0 0 0))
+  )
   (polyline (pts (xy 85.09 -85.09) (xy 176.53 -85.09))
     (stroke (width 0) (type default) (color 0 0 0 0))
@@
     (stroke (width 0) (type default) (color 0 0 0 0))
   )
+  (wire (pts (xy -26.67 90.17) (xy -26.67 88.9))
+    (stroke (width 0) (type default) (color 0 0 0 0))
+  )
   (wire (pts (xy 227.33 64.77) (xy 227.33 66.04))
     (stroke (width 0) (type default) (color 0 0 0 0))
@@
     (stroke (width 0) (type default) (color 0 0 0 0))
   )
+  (wire (pts (xy -19.05 85.09) (xy -19.05 74.93))
+    (stroke (width 0) (type default) (color 0 0 0 0))
+  )
   (polyline (pts (xy 283.21 -64.77) (xy 283.21 -62.23))
     (stroke (width 0) (type default) (color 0 0 0 0))
@@
     (stroke (width 0) (type default) (color 0 0 0 0))
   )
+  (wire (pts (xy -13.97 85.09) (xy -19.05 85.09))
+    (stroke (width 0) (type default) (color 0 0 0 0))
+  )
   (wire (pts (xy 374.65 73.66) (xy 374.65 72.39))
     (stroke (width 0) (type default) (color 0 0 0 0))
@@
     (stroke (width 0) (type default) (color 0 0 0 0))
   )
+  (wire (pts (xy -1.27 88.9) (xy -1.27 90.17))
+    (stroke (width 0) (type default) (color 0 0 0 0))
+  )
   (polyline (pts (xy 267.97 -53.34) (xy 283.21 -53.34))
     (stroke (width 0) (type default) (color 0 0 0 0))
@@
   )
   (polyline (pts (xy 176.53 -55.88) (xy 176.53 -44.45))
+    (stroke (width 0) (type default) (color 0 0 0 0))
+  )
+  (wire (pts (xy -19.05 74.93) (xy -13.97 74.93))
     (stroke (width 0) (type default) (color 0 0 0 0))
   )
@@
     (effects (font (size 1.27 1.27)) (justify left bottom))
   )
+  (text "12.5 == 1.05 + (cL1*cL2)/(cL1 + cL2)\n\n---------------------------------------\nResult: {12.44, {cL1 -> 22.79, cL2 -> 22.79}}\n"
+    (at -30.48 63.5 0)
+    (effects (font (size 1.27 1.27)) (justify left bottom))
+  )
   (text "GPIO 		Flash memory pin 	Solder bridge for memory use (default: shorted) 	Solder bridge for GPIO use (default: open)\n0.17 		CS 					SB13 												SB23\n0.19 		SCLK 				SB11 												SB21\n0.20 		SIO_0/SI 			SB12 												SB22\n0.21 		SIO_1/SO 			SB14 												SB24\n0.22 		SIO_2/WP 			SB15 												SB25\n0.23 		SIO_3/HOLD 			SB10 												SB20"
     (at 31.75 231.14 0)
@@
     (effects (font (size 1.27 1.27)) (justify left bottom))
   )
-  (text "f		32.000MHz +/- 10ppm\nESR		40${R}\nC_{L}		8pF\nD_{L}		100${mu}W\n\n"
-    (at 237.49 60.96 0)
+  (text "8 == 3 + (cL1*cL2)/(cL1 + cL2)\n\n---------------------------------------\nResult: {7.996, {cL1 -> 9.99, cL2 -> 9.992}}"
+    (at 236.22 50.8 0)
     (effects (font (size 1.27 1.27)) (justify left bottom))
   )
@@
   (label "ANT" (at 388.62 63.5 180)
     (effects (font (size 1.27 1.27)) (justify right bottom))
+  )
+  (symbol (lib_id "4ms_Power-symbol:GND") (at -26.67 90.17 0) (unit 1)
+    (in_bom yes) (on_board yes) (fields_autoplaced)
+    (property "Reference" "#PWR?" (id 0) (at -26.67 96.52 0)
+      (effects (font (size 1.27 1.27)) hide)
+    )
+    (property "Value" "GND" (id 1) (at -26.67 94.6134 0))
+    (property "Footprint" "" (id 2) (at -26.67 90.17 0)
+      (effects (font (size 1.27 1.27)) hide)
+    )
+    (property "Datasheet" "" (id 3) (at -26.67 90.17 0)
+      (effects (font (size 1.27 1.27)) hide)
+    )
+    (pin "1")
   )
   (symbol (lib_id "Device:C") (at 361.95 68.58 0) (unit 1)
@@
     (pin "1")
   )
-  (symbol (lib_id "1.Logic.Oscillators_Resonators:32.768kHz-ECS-0327-12.5-34B-TR") (at -1.27 67.31 0) (unit 1)
+  (symbol (lib_id "Device:C") (at -1.27 85.09 0) (unit 1)
+    (in_bom yes) (on_board yes) (fields_autoplaced)
+    (property "Reference" "C?" (id 0) (at 1.651 84.2553 0)
+      (effects (font (size 1.27 1.27)) (justify left))
+    )
+    (property "Value" "22.8pF, NP0, 1%" (id 1) (at 1.651 86.7922 0)
+      (effects (font (size 1.27 1.27)) (justify left))
+    )
+    (property "Footprint" "" (id 2) (at -0.3048 88.9 0)
+      (effects (font (size 1.27 1.27)) hide)
+    )
+    (property "Datasheet" "~" (id 3) (at -1.27 85.09 0)
+      (effects (font (size 1.27 1.27)) hide)
+    )
+    (pin "1")
+    (pin "2")
+  )
+  (symbol (lib_id "1.Logic.Oscillators_Resonators:32.768kHz-ECS-0327-12.5-34B-TR") (at -13.97 80.01 0) (unit 1)
     (in_bom yes) (on_board yes)
-    (property "Reference" "Y?" (id 0) (at 3.81 59.6931 0)
-      (effects (font (size 1.27 1.27)) (justify left))
-    )
-    (property "Value" "32.768kHz" (id 1) (at 3.81 62.23 0)
-      (effects (font (size 1.27 1.27)) (justify left))
-    )
-    (property "Footprint" "1.Logic.Oscillators:ECS-327-12-5-34B-TR" (id 2) (at -1.27 67.31 0)
-      (effects (font (size 1.27 1.27)) hide)
-    )
-    (property "Datasheet" "~" (id 3) (at -1.27 67.31 0)
+    (property "Reference" "Y?" (id 0) (at -8.89 72.3931 0)
+      (effects (font (size 1.27 1.27)) (justify left))
+    )
+    (property "Value" "32.768kHz" (id 1) (at -8.89 74.93 0)
+      (effects (font (size 1.27 1.27)) (justify left))
+    )
+    (property "Footprint" "1.Logic.Oscillators:ECS-327-12-5-34B-TR" (id 2) (at -13.97 80.01 0)
+      (effects (font (size 1.27 1.27)) hide)
+    )
+    (property "Datasheet" "~" (id 3) (at -13.97 80.01 0)
       (effects (font (size 1.27 1.27)) hide)
     )
@@
     (pin "2")
   )
-  (symbol (lib_id "Device:C") (at 262.89 20.32 0) (unit 1)
-    (in_bom yes) (on_board yes) (fields_autoplaced)
-    (property "Reference" "C?" (id 0) (at 265.811 19.4853 0)
-      (effects (font (size 1.27 1.27)) (justify left))
-    )
-    (property "Value" "C" (id 1) (at 265.811 22.0222 0)
-      (effects (font (size 1.27 1.27)) (justify left))
-    )
-    (property "Footprint" "" (id 2) (at 263.8552 24.13 0)
-      (effects (font (size 1.27 1.27)) hide)
-    )
-    (property "Datasheet" "~" (id 3) (at 262.89 20.32 0)
-      (effects (font (size 1.27 1.27)) hide)
-    )
-    (pin "1")
-    (pin "2")
+  (symbol (lib_id "4ms_Power-symbol:GND") (at -1.27 90.17 0) (unit 1)
+    (in_bom yes) (on_board yes) (fields_autoplaced)
+    (property "Reference" "#PWR?" (id 0) (at -1.27 96.52 0)
+      (effects (font (size 1.27 1.27)) hide)
+    )
+    (property "Value" "GND" (id 1) (at -1.27 94.6134 0))
+    (property "Footprint" "" (id 2) (at -1.27 90.17 0)
+      (effects (font (size 1.27 1.27)) hide)
+    )
+    (property "Datasheet" "" (id 3) (at -1.27 90.17 0)
+      (effects (font (size 1.27 1.27)) hide)
+    )
+    (pin "1")
+  )
+  (symbol (lib_id "4ms_Power-symbol:GND") (at -13.97 90.17 0) (unit 1)
+    (in_bom yes) (on_board yes) (fields_autoplaced)
+    (property "Reference" "#PWR?" (id 0) (at -13.97 96.52 0)
+      (effects (font (size 1.27 1.27)) hide)
+    )
+    (property "Value" "GND" (id 1) (at -13.97 94.6134 0))
+    (property "Footprint" "" (id 2) (at -13.97 90.17 0)
+      (effects (font (size 1.27 1.27)) hide)
+    )
+    (property "Datasheet" "" (id 3) (at -13.97 90.17 0)
+      (effects (font (size 1.27 1.27)) hide)
+    )
+    (pin "1")
   )
   (symbol (lib_id "0.Connectors:U.FL-R-SMT-110") (at 393.7 63.5 0) (unit 1)
@@
       (effects (font (size 1.27 1.27)) (justify left))
     )
-    (property "Value" "NP0 +-1%" (id 1) (at 230.251 62.6622 0)
+    (property "Value" "10pF, NP0, 0.1%" (id 1) (at 230.251 62.6622 0)
       (effects (font (size 1.27 1.27)) (justify left))
     )
@@
       (effects (font (size 1.27 1.27)) (justify left))
     )
-    (property "Value" "C" (id 1) (at 204.851 62.6622 0)
+    (property "Value" "10pF, NP0, 0.1%" (id 1) (at 204.851 62.6622 0)
       (effects (font (size 1.27 1.27)) (justify left))
     )
@@
     (pin "1")
   )
+  (symbol (lib_id "Device:C") (at -26.67 85.09 0) (unit 1)
+    (in_bom yes) (on_board yes) (fields_autoplaced)
+    (property "Reference" "C?" (id 0) (at -23.749 84.2553 0)
+      (effects (font (size 1.27 1.27)) (justify left))
+    )
+    (property "Value" "22.8pF, NP0, 1%" (id 1) (at -23.749 86.7922 0)
+      (effects (font (size 1.27 1.27)) (justify left))
+    )
+    (property "Footprint" "" (id 2) (at -25.7048 88.9 0)
+      (effects (font (size 1.27 1.27)) hide)
+    )
+    (property "Datasheet" "~" (id 3) (at -26.67 85.09 0)
+      (effects (font (size 1.27 1.27)) hide)
+    )
+    (pin "1")
+    (pin "2")
+  )
   (symbol (lib_id "Device:L") (at 349.25 63.5 90) (unit 1)

Commit message: NOR Flash
Parts:
- added C?: C, symbol Device:C
- added U?: W25Q128JVSS, Package_SO:SOIC-8_5.23x5.23mm_P1.27mm, symbol Memory_Flash:W25Q32JVSS
Connections:
- net GND: now also U?.4 (GND)
- new net +3V3: U?.8 (VCC)
- new net 0.17: U?.1 (~{CS})
- new net 0.19: U?.6 (CLK)
- new net 0.20: U?.5 (DI(IO0))
- new net 0.21: U?.2 (DO(IO1))
- new net 0.22: U?.3 (IO2)
- new net 0.23: U?.7 (IO3)
Other:
- note added: "FIXME: Decoupling capacitors"
- note removed: "GPIO Flash memory pin Solder bridge for memory use (default: shorted) Solder bridge for GPIO use (default: open) 0.17 CS SB13 SB23 0.19 SCLK SB11 SB21 0.20 SIO_0/SI SB12 SB22 0.21 SIO_1/SO SB14 SB24 0.22 SIO_2/WP SB15 SB25 0.23 SIO_3/HOLD SB10 SB20"
- note removed: "The memory is connected to the chip using the following GPIOs:"
Changed lines of the file:
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@@
   (junction (at -13.97 85.09) (diameter 0) (color 0 0 0 0)
   )
+  (wire (pts (xy 63.5 243.84) (xy 38.1 243.84))
+    (stroke (width 0) (type default) (color 0 0 0 0))
+  )
+  (wire (pts (xy 38.1 241.3) (xy 63.5 241.3))
+    (stroke (width 0) (type default) (color 0 0 0 0))
+  )
+  (wire (pts (xy 127 261.62) (xy 124.46 261.62))
+    (stroke (width 0) (type default) (color 0 0 0 0))
+  )
   (polyline (pts (xy 100.33 -41.91) (xy 85.09 -41.91))
     (stroke (width 0) (type default) (color 0 0 0 0))
@@
     (stroke (width 0) (type default) (color 0 0 0 0))
   )
+  (wire (pts (xy 127 254) (xy 124.46 254))
+    (stroke (width 0) (type default) (color 0 0 0 0))
+  )
   (wire (pts (xy -26.67 80.01) (xy -26.67 81.28))
     (stroke (width 0) (type default) (color 0 0 0 0))
@@
     (stroke (width 0) (type default) (color 0 0 0 0))
   )
+  (wire (pts (xy 111.76 243.84) (xy 111.76 248.92))
+    (stroke (width 0) (type default) (color 0 0 0 0))
+  )
+  (wire (pts (xy 63.5 254) (xy 38.1 254))
+    (stroke (width 0) (type default) (color 0 0 0 0))
+  )
   (wire (pts (xy 214.63 60.96) (xy 209.55 60.96))
     (stroke (width 0) (type default) (color 0 0 0 0))
@@
     (stroke (width 0) (type default) (color 0 0 0 0))
   )
+  (wire (pts (xy 96.52 261.62) (xy 99.06 261.62))
+    (stroke (width 0) (type default) (color 0 0 0 0))
+  )
+  (wire (pts (xy 63.5 251.46) (xy 38.1 251.46))
+    (stroke (width 0) (type default) (color 0 0 0 0))
+  )
   (wire (pts (xy 374.65 63.5) (xy 381 63.5))
     (stroke (width 0) (type default) (color 0 0 0 0))
@@
     (stroke (width 0) (type default) (color 0 0 0 0))
   )
+  (wire (pts (xy 63.5 256.54) (xy 38.1 256.54))
+    (stroke (width 0) (type default) (color 0 0 0 0))
+  )
+  (wire (pts (xy 111.76 276.86) (xy 111.76 269.24))
+    (stroke (width 0) (type default) (color 0 0 0 0))
+  )
   (polyline (pts (xy 176.53 -85.09) (xy 176.53 -74.93))
     (stroke (width 0) (type default) (color 0 0 0 0))
   )
+  (wire (pts (xy 63.5 248.92) (xy 38.1 248.92))
+    (stroke (width 0) (type default) (color 0 0 0 0))
+  )
   (wire (pts (xy 330.2 72.39) (xy 336.55 72.39))
     (stroke (width 0) (type default) (color 0 0 0 0))
@@
     (stroke (width 0) (type default) (color 0 0 0 0))
   )
+  (wire (pts (xy 96.52 256.54) (xy 99.06 256.54))
+    (stroke (width 0) (type default) (color 0 0 0 0))
+  )
   (polyline (pts (xy 184.15 -72.39) (xy 208.28 -69.85))
     (stroke (width 0) (type default) (color 0 0 0 0))
   )
+  (wire (pts (xy 127 256.54) (xy 124.46 256.54))
+    (stroke (width 0) (type default) (color 0 0 0 0))
+  )
   (polyline (pts (xy 232.41 -69.85) (xy 217.17 -68.58))
     (stroke (width 0) (type default) (color 0 0 0 0))
@@
     (stroke (width 0) (type default) (color 0 0 0 0))
   )
+  (wire (pts (xy 127 264.16) (xy 124.46 264.16))
+    (stroke (width 0) (type default) (color 0 0 0 0))
+  )
   (polyline (pts (xy 147.32 -29.21) (xy 147.32 -17.78))
     (stroke (width 0) (type default) (color 0 0 0 0))
@@
   )
   (text "Analog SW" (at 142.24 -48.26 0)
-    (effects (font (size 1.27 1.27)) (justify left bottom))
-  )
-  (text "The memory is connected to the chip using the following GPIOs:"
-    (at 29.21 208.28 0)
     (effects (font (size 1.27 1.27)) (justify left bottom))
   )
@@
     (effects (font (size 1.27 1.27)) (justify left bottom))
   )
-  (text "GPIO 		Flash memory pin 	Solder bridge for memory use (default: shorted) 	Solder bridge for GPIO use (default: open)\n0.17 		CS 					SB13 												SB23\n0.19 		SCLK 				SB11 												SB21\n0.20 		SIO_0/SI 			SB12 												SB22\n0.21 		SIO_1/SO 			SB14 												SB24\n0.22 		SIO_2/WP 			SB15 												SB25\n0.23 		SIO_3/HOLD 			SB10 												SB20"
-    (at 31.75 231.14 0)
-    (effects (font (size 1.27 1.27)) (justify left bottom))
-  )
   (text "External\nQSPI Flash" (at 233.68 -60.96 0)
     (effects (font (size 1.27 1.27)) (justify left bottom))
@@
     (effects (font (size 1.27 1.27)) (justify left bottom))
   )
+  (text "FIXME: Decoupling capacitors" (at 140.97 240.03 0)
+    (effects (font (size 1.27 1.27)) (justify left bottom))
+  )
   (text "32 MHz \nOscillator" (at 233.68 -43.18 0)
     (effects (font (size 1.27 1.27)) (justify left bottom))
@@
   )
   (text " The nRF52840 DK has a 64 Mb external flash memory. The memory is a multi-I/O memory supporting both regular SPI and Quad SPI. "
-    (at 26.67 196.85 0)
+    (at 29.21 234.95 0)
     (effects (font (size 1.27 1.27)) (justify left bottom))
   )
@@
     (effects (font (size 1.27 1.27)) (justify left bottom))
   )
+  (label "FLASH_{SIO1}" (at 127 256.54 0)
+    (effects (font (size 1.27 1.27)) (justify left bottom))
+  )
+  (label "FLASH_{SIO3}" (at 127 264.16 0)
+    (effects (font (size 1.27 1.27)) (justify left bottom))
+  )
+  (label "0.20" (at 63.5 248.92 0)
+    (effects (font (size 1.27 1.27)) (justify left bottom))
+  )
+  (label "0.22" (at 63.5 254 0)
+    (effects (font (size 1.27 1.27)) (justify left bottom))
+  )
+  (label "FLASH_{~{CS}}" (at 96.52 256.54 180)
+    (effects (font (size 1.27 1.27)) (justify right bottom))
+  )
+  (label "FLASH_{SIO0}" (at 127 254 0)
+    (effects (font (size 1.27 1.27)) (justify left bottom))
+  )
+  (label "FLASH_{SCLK}" (at 96.52 261.62 180)
+    (effects (font (size 1.27 1.27)) (justify right bottom))
+  )
+  (label "FLASH_{SIO0}" (at 38.1 248.92 180)
+    (effects (font (size 1.27 1.27)) (justify right bottom))
+  )
+  (label "FLASH_{SIO1}" (at 38.1 251.46 180)
+    (effects (font (size 1.27 1.27)) (justify right bottom))
+  )
+  (label "FLASH_{SIO3}" (at 38.1 256.54 180)
+    (effects (font (size 1.27 1.27)) (justify right bottom))
+  )
+  (label "0.23" (at 63.5 256.54 0)
+    (effects (font (size 1.27 1.27)) (justify left bottom))
+  )
+  (label "0.21" (at 63.5 251.46 0)
+    (effects (font (size 1.27 1.27)) (justify left bottom))
+  )
+  (label "FLASH_{SIO2}" (at 38.1 254 180)
+    (effects (font (size 1.27 1.27)) (justify right bottom))
+  )
+  (label "FLASH_{~{CS}}" (at 38.1 241.3 180)
+    (effects (font (size 1.27 1.27)) (justify right bottom))
+  )
   (label "RF" (at 381 63.5 0)
     (effects (font (size 1.27 1.27)) (justify left bottom))
   )
+  (label "0.17" (at 63.5 241.3 0)
+    (effects (font (size 1.27 1.27)) (justify left bottom))
+  )
+  (label "FLASH_{SIO2}" (at 127 261.62 0)
+    (effects (font (size 1.27 1.27)) (justify left bottom))
+  )
   (label "ANT" (at 388.62 63.5 180)
+    (effects (font (size 1.27 1.27)) (justify right bottom))
+  )
+  (label "0.19" (at 63.5 243.84 0)
+    (effects (font (size 1.27 1.27)) (justify left bottom))
+  )
+  (label "FLASH_{SCLK}" (at 38.1 243.84 180)
     (effects (font (size 1.27 1.27)) (justify right bottom))
   )
@@
     (pin "1")
     (pin "2")
+  )
+  (symbol (lib_id "4ms_Power-symbol:+3.3V") (at 111.76 243.84 0) (unit 1)
+    (in_bom yes) (on_board yes) (fields_autoplaced)
+    (property "Reference" "#PWR?" (id 0) (at 111.76 247.65 0)
+      (effects (font (size 1.27 1.27)) hide)
+    )
+    (property "Value" "+3.3V" (id 1) (at 111.76 240.2642 0))
+    (property "Footprint" "" (id 2) (at 111.76 243.84 0)
+      (effects (font (size 1.27 1.27)) hide)
+    )
+    (property "Datasheet" "" (id 3) (at 111.76 243.84 0)
+      (effects (font (size 1.27 1.27)) hide)
+    )
+    (pin "1")
   )
   (symbol (lib_id "4ms_Power-symbol:GND") (at 361.95 73.66 0) (unit 1)
@@
     (pin "4")
   )
+  (symbol (lib_id "4ms_Power-symbol:GND") (at 111.76 276.86 0) (unit 1)
+    (in_bom yes) (on_board yes) (fields_autoplaced)
+    (property "Reference" "#PWR?" (id 0) (at 111.76 283.21 0)
+      (effects (font (size 1.27 1.27)) hide)
+    )
+    (property "Value" "GND" (id 1) (at 111.76 281.3034 0))
+    (property "Footprint" "" (id 2) (at 111.76 276.86 0)
+      (effects (font (size 1.27 1.27)) hide)
+    )
+    (property "Datasheet" "" (id 3) (at 111.76 276.86 0)
+      (effects (font (size 1.27 1.27)) hide)
+    )
+    (pin "1")
+  )
   (symbol (lib_id "4ms_Power-symbol:GND") (at 393.7 73.66 0) (unit 1)
     (in_bom yes) (on_board yes) (fields_autoplaced)
@@
     )
     (property "Datasheet" "~" (id 3) (at -1.27 85.09 0)
+      (effects (font (size 1.27 1.27)) hide)
+    )
+    (pin "1")
+    (pin "2")
+  )
+  (symbol (lib_id "Device:C") (at 137.16 243.84 0) (unit 1)
+    (in_bom yes) (on_board yes) (fields_autoplaced)
+    (property "Reference" "C?" (id 0) (at 140.081 243.0053 0)
+      (effects (font (size 1.27 1.27)) (justify left))
+    )
+    (property "Value" "C" (id 1) (at 140.081 245.5422 0)
+      (effects (font (size 1.27 1.27)) (justify left))
+    )
+    (property "Footprint" "" (id 2) (at 138.1252 247.65 0)
+      (effects (font (size 1.27 1.27)) hide)
+    )
+    (property "Datasheet" "~" (id 3) (at 137.16 243.84 0)
       (effects (font (size 1.27 1.27)) hide)
     )
@@
     (pin "1")
   )
+  (symbol (lib_id "Memory_Flash:W25Q32JVSS") (at 111.76 259.08 0) (unit 1)
+    (in_bom yes) (on_board yes) (fields_autoplaced)
+    (property "Reference" "U?" (id 0) (at 120.5112 247.7602 0))
+    (property "Value" "W25Q128JVSS" (id 1) (at 120.5112 250.2971 0))
+    (property "Footprint" "Package_SO:SOIC-8_5.23x5.23mm_P1.27mm" (id 2) (at 111.76 259.08 0)
+      (effects (font (size 1.27 1.27)) hide)
+    )
+    (property "Datasheet" "http://www.winbond.com/resource-files/w25q32jv%20revg%2003272018%20plus.pdf" (id 3) (at 111.76 259.08 0)
+      (effects (font (size 1.27 1.27)) hide)
+    )
+    (pin "1")
+    (pin "2")
+    (pin "3")
+    (pin "4")
+    (pin "5")
+    (pin "6")
+    (pin "7")
+    (pin "8")
+  )
   (symbol (lib_id "4ms_Power-symbol:GND") (at 227.33 66.04 0) (unit 1)
