File: hw/nrf_mcu.kicad_sch (KiCad schematic)
At the start: 14 parts

Commit message: Cypress USB interface symbol & Layout needs fixing
Connections:
- net ANT: now also C?.1, C?.1, L?.2
- net RF: now also C?.1, L?.1; no longer C?.1, C?.1, L?.2
Other:
- note added: "* Decoupling & Power * SWD/JTAG? * Reset/boot btn * GPIO header * GPIO mappings? (Section 7) * Ordering codes & Variations? * Fault detection circuitry * USB Interfacing? * Interface with RP2040? * Interface with CYP EZPD?"
- note removed: "* USB IO? * SWD/JTAG? * NFC? * GPIO mappings? (Section 7) * Flash memory (QSPI)? * Ordering codes & Variations?"
- moved on the sheet: C?, J?, L?, U?, Y?
