File: hw/nrf_mcu.kicad_sch (KiCad schematic)
At the start: 14 parts

Commit message: lolz
Parts:
- removed C?: 0.5pF, symbol Device:C
- removed C?: DNP, symbol Device:C
- removed C? (x2): 22.8pF, NP0, 1%, symbol Device:C
- removed C?: C, symbol Device:C
- removed C?: 0.8pF, symbol Device:C
- removed C? (x2): 10pF, NP0, 0.1%, symbol Device:C
- removed J?: U.FL-R-SMT-110, CONN_U.FL-R-SMT-110_HIR, symbol 0.Connectors:U.FL-R-SMT-110
- removed L?: 4.7nH, symbol Device:L
- removed U?: W25Q128JVSS, Package_SO:SOIC-8_5.23x5.23mm_P1.27mm, symbol Memory_Flash:W25Q32JVSS
- removed U?: nRF52840-QAAA, Package_DFN_QFN:Nordic_AQFN-73-1EP_7x7mm_P0.5mm, symbol 1.Embedded.Microcontrollers:nRF52840-QAAA
- removed Y?: 32.000MHz, 1.Logic.Oscillators:32MHz-ECS-320-8-37B2-7KM-TR, symbol 1.Logic.Oscillators_Resonators:32MHz-ECS-320-8-37B2-7KM-TR
- removed Y?: 32.768kHz, 1.Logic.Oscillators:ECS-327-12-5-34B-TR, symbol 1.Logic.Oscillators_Resonators:32.768kHz-ECS-0327-12.5-34B-TR
Other:
- note removed: "* Decoupling & Power * SWD/JTAG? * Reset/boot btn * GPIO header * GPIO mappings? (Section 7) * Ordering codes & Variations? * Fault detection circuitry * USB Interfacing? * Interface with RP2040? * Interface with CYP EZPD?"
- note removed: "12.5 == 1.05 + (cL1*cL2)/(cL1 + cL2) --------------------------------------- Result: {12.44, {cL1 -> 22.79, cL2 -> 22.79}}"
- note removed: "32 MHz Oscillator"
- note removed: "32.768kHz Oscillator"
- note removed: "8 == 3 + (cL1*cL2)/(cL1 + cL2) --------------------------------------- Result: {7.996, {cL1 -> 9.99, cL2 -> 9.992}}"
- note removed: "Analog SW"
- note removed: "Battery"
- note removed: "Buttons"
- note removed: "Current Measurement"
- note removed: "Debug In"
- note removed: "Debug Out"
- note removed: "Ext. PSU"
- note removed: "External QSPI Flash"
- note removed: "FIXME: Decoupling capacitors"
- note removed: "GPIO"
- note removed: "IF Boot/Reset"
- note removed: "IF MCU USB"
- note removed: "Interface MCU"
- note removed: "LEDs"
- note removed: "Li-Ion"
- note removed: "Power Supply"
- note removed: "Power Sw"
- note removed: "RF Connector"
- note removed: "RF Matching Network"
- note removed: "The nRF52840 DK has a 64 Mb external flash memory. The memory is a multi-I/O memory supporting both regular SPI and Quad SPI."
- note removed: "four-component RF match is recommended for new designs"
- note removed: "nRF Power Source SW"
- note removed: "nRF USB"
- note removed: "nRF52840"
