File: hw/friendly-keyboard.kicad_pcb (KiCad board)
At the start: 4 copper layers, 56 x 56 mm, 5 parts

Commit message: lolz
Parts:
- removed LOGO**: 1_wordmark, 0:1_wordmark
- removed M_BL, M_BR, M_TL, M_TR: MountingHole_3.2mm_M3_ISO14580, MountingHole:MountingHole_3.2mm_M3_ISO14580
- added C10: 10μF, Capacitor_Tantalum_SMD:CP_EIA-2012-15_AVX-P, F.Cu at (212.1, 95.7)
- added C11: 22μF, Capacitor_Tantalum_SMD:CP_EIA-2012-15_AVX-P, F.Cu at (205.8, 101.7)
- added C12: 100nF, Capacitor_SMD:C_0201_0603Metric, F.Cu at (232.2, 90.6)
- added C13: 2.2μF, Capacitor_SMD:C_0201_0603Metric, F.Cu at (237.2, 88.1)
- added C14: 10μF, Capacitor_SMD:C_0201_0603Metric, F.Cu at (223.1, 103.0)
- added C15: 10μF, Capacitor_SMD:C_0201_0603Metric, F.Cu at (239.6, 87.6)
- added C16: 10μF, Capacitor_Tantalum_SMD:CP_EIA-2012-15_AVX-P, F.Cu at (200.5, 107.0)
- added C17: 100nF, Capacitor_SMD:C_0201_0603Metric, F.Cu at (231.3, 97.6)
- added C18: 100nF, Capacitor_SMD:C_0201_0603Metric, F.Cu at (223.1, 101.2)
- added C19: 1μF, Capacitor_SMD:C_0201_0603Metric, F.Cu at (220.2, 104.0)
- added C20: 1μF, Capacitor_SMD:C_0603_1608Metric, F.Cu at (227.0, 89.2)
- added C21: 2.2nF, Capacitor_SMD:C_0201_0603Metric, F.Cu at (234.1, 94.1)
- added C22: 2.2nF, Capacitor_SMD:C_0201_0603Metric, F.Cu at (226.4, 98.4)
- added C23: 1μF, Capacitor_SMD:C_0603_1608Metric, F.Cu at (225.1, 94.5)
- added C24: 4.7μF, Capacitor_SMD:C_0805_2012Metric, F.Cu at (217.2, 91.4)
- added C25: 4.7μF, Capacitor_SMD:C_0805_2012Metric, F.Cu at (222.8, 86.2)
- added C26: 100nF, Capacitor_SMD:C_0201_0603Metric, F.Cu at (228.8, 95.9)
- added C27: 100nF, Capacitor_SMD:C_0201_0603Metric, F.Cu at (232.2, 92.4)
- added C28: 100nF, Capacitor_SMD:C_0201_0603Metric, F.Cu at (228.8, 99.4)
- added C29: 10μF, Capacitor_SMD:C_0805_2012Metric, F.Cu at (205.0, 107.1)
- added C3: 100nF, Capacitor_SMD:C_0201_0603Metric, F.Cu at (225.6, 101.9)
- added C30: 1.2pF, Capacitor_SMD:C_0201_0603Metric, F.Cu at (239.6, 89.3)
- added C31: DNP, Capacitor_SMD:C_0201_0603Metric, F.Cu at (225.6, 103.7)
- added C32: 1.8pF, Capacitor_SMD:C_0201_0603Metric, F.Cu at (219.3, 106.0)
- added C33: 9.5pF, Capacitor_SMD:C_0201_0603Metric, F.Cu at (241.2, 85.6)
- added C34: 0.7pF, Capacitor_SMD:C_0201_0603Metric, F.Cu at (216.7, 108.2)
- added C35: DNP, Capacitor_SMD:C_0201_0603Metric, F.Cu at (214.2, 108.7)
- added C36: 1.2pF, Capacitor_SMD:C_0201_0603Metric, F.Cu at (237.2, 89.8)
- added C37: DNP, Capacitor_SMD:C_0201_0603Metric, F.Cu at (234.7, 90.1)
- added C38: 1.8pF, Capacitor_SMD:C_0201_0603Metric, F.Cu at (221.8, 105.7)
- added C39: 9.5pF, Capacitor_SMD:C_0201_0603Metric, F.Cu at (234.7, 91.8)
- added C4: 100nF, Capacitor_SMD:C_0201_0603Metric, F.Cu at (231.6, 94.1)
- added C40: C, Capacitor_SMD:C_0402_1005Metric, F.Cu at (238.5, 85.7)
- added C41: C, Capacitor_SMD:C_0402_1005Metric, F.Cu at (234.5, 88.2)
- added C42: 1pF, Capacitor_SMD:C_0201_0603Metric, F.Cu at (226.4, 96.7)
- added C5: 100nF, Capacitor_SMD:C_0201_0603Metric, F.Cu at (237.1, 91.6)
- added C6: 100nF, Capacitor_SMD:C_0201_0603Metric, F.Cu at (221.8, 107.5)
- added C7: 100nF, Capacitor_SMD:C_0201_0603Metric, F.Cu at (231.6, 95.9)
- added C8: 100nF, Capacitor_SMD:C_0201_0603Metric, F.Cu at (225.8, 100.2)
- added C9: 2.2μF, Capacitor_SMD:C_0603_1608Metric, F.Cu at (209.2, 106.6)
- added D2: LED_Filled, LED_SMD:LED_0805_2012Metric, F.Cu at (222.8, 89.2)
- added J2: USB_C_Receptacle_USB2.0, Connector_USB:USB_C_Receptacle_Palconn_UTC16-G, F.Cu at (159.0, 154.9)
- added L1: 10μH, 1.Inductors.L_SRN_LAB2:L_SRN_2016_2010-1R0M, F.Cu at (227.2, 86.3)
- added L2: 0.47μH, 1.Inductors.L_SRN_LAB2:L_SRN_2016_2012-R47M, F.Cu at (211.8, 98.7)
- added L3: 10μH, 1.Inductors.L_SRN_LAB2:L_SRN_2016_2010-1R0M, F.Cu at (217.2, 94.5)
- added L4: 1.9nH, Inductor_SMD:L_0402_1005Metric, F.Cu at (217.5, 102.1)
- added L5: NC, Inductor_SMD:L_0402_1005Metric, F.Cu at (217.5, 104.1)
- added L6: 2.2nH, Inductor_SMD:L_0402_1005Metric, F.Cu at (228.9, 94.0)
- added L7: 1.9nH, Inductor_SMD:L_0402_1005Metric, F.Cu at (205.0, 104.1)
- added L8: NC, Inductor_SMD:L_0402_1005Metric, F.Cu at (216.7, 106.3)
- added Q1: ?, Package_TO_SOT_SMD:SOT-23-5, F.Cu at (218.0, 86.9)
- added Q2: ?, Package_TO_SOT_SMD:SOT-23-5, F.Cu at (212.4, 92.1)
- added R1: 2.2Ω, Resistor_SMD:R_0603_1608Metric, F.Cu at (221.4, 92.0)
- added R10: 470Ω, Resistor_SMD:R_0603_1608Metric, F.Cu at (210.1, 104.1)
- added R11: 100kΩ, Resistor_SMD:R_0603_1608Metric, F.Cu at (215.6, 98.4)
- added R12: R, Resistor_SMD:R_0603_1608Metric, F.Cu at (231.1, 88.5)
- added R13: 100kΩ, Resistor_SMD:R_0603_1608Metric, F.Cu at (214.1, 101.6)
- added R14: R, Resistor_SMD:R_0603_1608Metric, F.Cu at (213.2, 106.6)
- added R15: 100kΩ, Resistor_SMD:R_0603_1608Metric, F.Cu at (214.1, 104.1)
- added R16: 1MΩ, Resistor_SMD:R_0603_1608Metric, F.Cu at (219.6, 99.8)
- added R17: RITOPOFF, Resistor_SMD:R_0603_1608Metric, F.Cu at (219.6, 97.3)
- added R18: R, Resistor_SMD:R_0603_1608Metric, F.Cu at (231.1, 86.0)
- added R2: 0Ω, Resistor_SMD:R_0603_1608Metric, F.Cu at (225.5, 92.0)
- added R3: 49.9Ω, Resistor_SMD:R_0402_1005Metric, F.Cu at (208.7, 108.8)
- added R4: 28Ω, Resistor_SMD:R_0402_1005Metric, F.Cu at (220.4, 102.1)
- added R5: 28Ω, Resistor_SMD:R_0402_1005Metric, F.Cu at (211.6, 108.8)
- added R6: 0Ω, Resistor_SMD:R_0603_1608Metric, F.Cu at (210.1, 101.6)
- added R7: 49.9Ω, Resistor_SMD:R_0402_1005Metric, F.Cu at (223.1, 99.4)
- added R8: CONFIG, Resistor_SMD:R_0603_1608Metric, F.Cu at (235.1, 86.0)
- added TH1: Thermistor, Resistor_SMD:R_0603_1608Metric, F.Cu at (221.1, 94.5)
- added U2: MAX9027EBT+T, 0:MAX9027EBT-T, F.Cu at (211.9, 140.4)
- added U3: NRF5340-CLAA-R, 1.Embedded.Specialized:NRF5340-CLAA-R, F.Cu at (199.7, 153.3)
- added U4: NRF21540-QDAA-R, Package_DFN_QFN:QFN-16-1EP_3x3mm_P0.5mm_EP1.75x1.75mm, F.Cu at (201.9, 159.1)
- added U5: MAX77751CEFG+, 1.Power.BattMgmt:MAX77751CEFG+, F.Cu at (207.7, 146.3)
- added U6: MAX9027EBT+T, 0:MAX9027EBT-T, F.Cu at (211.9, 142.9)
Other:
- board size 56 x 56 mm -> 18 x 35 mm
- copper layers 4 -> 6
- rule pad_to_mask_clearance: 0.0762 -> 0
