File: hw/friendly-keyboard.kicad_sch (KiCad schematic)
At the start: 2 parts

Commit message: lolz
Parts:
- removed U?: CY8C9540, 1.Logic.IO_Expanders:CY8C9540A-24PVXI, symbol 1.Logic.IO_Expanders:CY8C9540
- removed U?: RP2040, Package_DFN_QFN:QFN-56-1EP_7x7mm_P0.4mm_EP3.2x3.2mm, symbol MCU_RaspberryPi:RP2040
- added AE1, AE2: Antenna, symbol Device:Antenna
- added BT1: Batt, Connector_JST:JST_EH_S2B-EH_1x02_P2.50mm_Horizontal, symbol Device:Battery_Cell
- added C10, C16: 10${uF}, Capacitor_Tantalum_SMD:CP_EIA-2012-15_AVX-P, symbol Device:C_Polarized_US
- added C11: 22${uF}, Capacitor_Tantalum_SMD:CP_EIA-2012-15_AVX-P, symbol Device:C_Polarized_US
- added C12, C17, C18, C26, C27, C28, C3, C4, C5, C6, C7, C8: 100nF, Capacitor_SMD:C_0201_0603Metric, symbol Device:C
- added C13: 2.2${uF}, Capacitor_SMD:C_0201_0603Metric, symbol Device:C
- added C14, C15: 10${uF}, Capacitor_SMD:C_0201_0603Metric, symbol Device:C
- added C19: 1${uF}, Capacitor_SMD:C_0201_0603Metric, symbol Device:C
- added C20, C23: 1${uF}, Capacitor_SMD:C_0603_1608Metric, symbol Device:C
- added C21, C22: 2.2nF, Capacitor_SMD:C_0201_0603Metric, symbol Device:C
- added C24, C25: 4.7${uF}, Capacitor_SMD:C_0805_2012Metric, symbol Device:C
- added C29: 10${uF}, Capacitor_SMD:C_0805_2012Metric, symbol Device:C
- added C30, C36: 1.2pF, Capacitor_SMD:C_0201_0603Metric, symbol Device:C
- added C31, C35, C37: DNP, Capacitor_SMD:C_0201_0603Metric, symbol Device:C
- added C32, C38: 1.8pF, Capacitor_SMD:C_0201_0603Metric, symbol Device:C
- added C33, C39: 9.5pF, Capacitor_SMD:C_0201_0603Metric, symbol Device:C
- added C34: 0.7pF, Capacitor_SMD:C_0201_0603Metric, symbol Device:C
- added C40, C41: C, Capacitor_SMD:C_0402_1005Metric, symbol Device:C
- added C42: 1pF, Capacitor_SMD:C_0201_0603Metric, symbol Device:C
- added C9: 2.2${uF}, Capacitor_SMD:C_0603_1608Metric, symbol Device:C
- added C?: 10pF, symbol Device:C
- added D2: LED_Filled, LED_SMD:LED_0805_2012Metric, symbol Device:LED_Filled
- added J2: USB_C_Receptacle_USB2.0, Connector_USB:USB_C_Receptacle_Palconn_UTC16-G, symbol Connector:USB_C_Receptacle_USB2.0
- added L1, L3: 10${uh}, 1.Inductors.L_SRN_LAB2:L_SRN_2016_2010-1R0M, symbol Device:L
- added L2: 0.47${uh}, 1.Inductors.L_SRN_LAB2:L_SRN_2016_2012-R47M, symbol 1.Inductors.L_SRN_LAB2:L_SRN_2016_2010-R47M
- added L4, L7: 1.9nH, Inductor_SMD:L_0402_1005Metric, symbol Device:L
- added L5, L8: NC, Inductor_SMD:L_0402_1005Metric, symbol Device:L
- added L6: 2.2nH, Inductor_SMD:L_0402_1005Metric, symbol Device:L
- added Q1, Q2: ?, Package_TO_SOT_SMD:SOT-23-5, symbol 4ms_Transistor:PMOS_IRF5305PBF
- added R1: 2.2${R}, Resistor_SMD:R_0603_1608Metric, symbol Device:R
- added R10: 470${R}, Resistor_SMD:R_0603_1608Metric, symbol Device:R
- added R11, R13, R15: 100${kR}, Resistor_SMD:R_0603_1608Metric, symbol Device:R
- added R12, R14, R18: R, Resistor_SMD:R_0603_1608Metric, symbol Device:R
- added R16: 1M${R}, Resistor_SMD:R_0603_1608Metric, symbol Device:R
- added R17: RITOPOFF, Resistor_SMD:R_0603_1608Metric, symbol Device:R
- added R2, R6: 0${R}, Resistor_SMD:R_0603_1608Metric, symbol Device:R
- added R3, R7: 49.9${R}, Resistor_SMD:R_0402_1005Metric, symbol Device:R
- added R4, R5: 28${R}, Resistor_SMD:R_0402_1005Metric, symbol Device:R
- added R8: CONFIG, Resistor_SMD:R_0603_1608Metric, symbol Device:R
- added R?: R_Shunt, Resistor_SMD:R_Shunt_Ohmite_LVK12, symbol Device:R_Shunt
- added R?: 1M${R, symbol Device:R
- added TH1: Thermistor, Resistor_SMD:R_0603_1608Metric, symbol Device:Thermistor
- added TIE1, TIE?: NetTie, 4ms_SolderJumper:Net_Tie_0.16mm_6mil, symbol 4ms_Net-tie:NetTie
- added U2, U6: MAX9027EBT+T, 0:MAX9027EBT-T, symbol 0.Project:MAX9027EBT+T
- added U3: NRF5340-CLAA-R, 1.Embedded.Specialized:NRF5340-CLAA-R, symbol 1.Embedded.Specialized:NRF5340-CLAA-R
- added U4: NRF21540-QDAA-R, Package_DFN_QFN:QFN-16-1EP_3x3mm_P0.5mm_EP1.75x1.75mm, symbol 1.Communications.Amplifiers:NRF21540-QDAA-R
- added U5: MAX77751CEFG+, 1.Power.BattMgmt:MAX77751CEFG+, symbol 0.Project:MAX77751CEFG+
- added Y1: 32MHz-ECS-320-8-37B2-7KM-TR, 1.Logic.Oscillators:32MHz-ECS-320-8-37B2-7KM-TR, symbol 1.Logic.Oscillators_Resonators:32MHz-ECS-320-8-37B2-7KM-TR
Connections:
- new net: C26.1, U3.B5 (DECN)
- new net: C34.1, L6.1, U3.D1 (ANT)
- new net: C13.1, U5.17 (PVL)
- new net: AE1.1 (A), C32.2, C33.2, R2.2
- new net: C36.2, C37.2, L7.2, L8.2, R6.1, R7.1
- new net: C12.2, L2.1, U5.20 (LX), U5.21 (LX)
- new net: BT1.2 (-), R?.1
- new net: R8.1, U5.12 (IFAST)
- new net: AE2.1 (A), C38.2, C39.2, R6.2
- new net: C23.1, L3.1, U3.A7 (DECD)
- new net: C40.1, U3.A2 (XC2), Y1.1
- new net: C41.1, U3.A1 (XC1), Y1.3
- new net: R15.1, U6.A2
- new net: C25.1, U3.C11 (DECUSB)
- new net: R14.2, R18.1, U6.B1 (+)
- new net: C20.1, C21.1, L1.1, U3.B1 (DECRF), U3.B4 (DECR)
- new net: C24.1, R1.2, U3.B11 (VBUS)
- new net: L1.2, U3.B6 (DCCR)
- new net: C28.1, C29.1
- new net: R11.2, TH1.1, U2.B1 (+), U6.B3 (-)
- new net: R4.2, U3.A11 (D-)
- new net: C10.1, C11.1, U5.22 (BYP)
- new net: C?.1, J2.S1 (SHIELD), R?.1
- new net: C30.2, C31.2, L4.2, L5.2, R2.1, R3.1
- new net: L7.1, U4.3 (ANT2)
- new net: R12.2, R14.1, U2.B3 (-)
- new net: L4.1, U4.2 (ANT1)
- new net: R5.2, U3.A12 (D+)
- new net: C12.1, U5.1 (BST)
- new net: R13.1, U2.A2
- new net: D2.2 (A), R10.2
- new net: C42.2, U4.10 (TRX)
- new net: C27.1, U3.B8 (DECA)
- new net: C19.1, U3.B7 (VDD)
- new net: L3.2, U3.A9 (DCCD)
- new net: C22.1, U3.B10 (VDD)
- new net: U3.B12 (VDDH), U3.E11 (VDD)
- new net +5V: C14.1, C15.1, L2.2, R10.1, R11.1, R12.1, U2.A1 (V+), U5.15 (SYS), U5.16 (SYS), U6.A1 (V+)
- new net +BATT: BT1.1 (+), C16.1, U5.13 (BATT), U5.14 (BATT)
- new net ANT_SEL: U4.8 (ANT_SEL)
- new net AVSS: C17.2, C18.2, C19.2, C20.2, C21.2, C22.2, C23.2, C24.2, C25.2, C26.2, C27.2, C28.2, C29.2, C3.2, C30.1, C31.1, C32.1, C33.1, C34.2, C35.2, C36.1, C37.1, C38.1, C39.1, C4.2, C40.2, C41.2, C5.2, C6.2, C7.2, C8.2, C9.2, C?.2, J2.A1 (GND), J2.A12 (GND), J2.B1 (GND), J2.B12 (GND), L5.1, L8.1, Q1.3 (S), Q2.3 (S), R16.2, R17.2, R18.2, R3.2, R7.2, R8.2, R?.2, TH1.2, U2.A3 (V-), U2.B2 (V-), U3.A5 (VSS), U3.B2 (VSS), U3.B9 (VSS), U3.C2 (VSS), U3.D12 (VSS), U3.E5 (VSS), U3.E6 (VSS), U3.E7 (VSS), U3.E8 (VSS), U3.F5 (VSS), U3.F6 (VSS), U3.F7 (VSS), U3.F8 (VSS), U3.G5 (AVSS), U3.G6 (VSS), U3.G7 (VSS), U3.G8 (VSS), U3.K11 (AVSS), U3.K6 (AVSS), U4.1 (VSS), U4.16 (VSS), U4.17 (VSS), U5.8 (ENBST), U5.9 (GND), U6.A3 (V-), U6.B2 (V-), Y1.2, Y1.4
- new net CHARGE_STAT: U5.3 (STAT)
- new net GNDPWR: C10.2, C11.2, C13.2, C14.2, C15.2, C16.2, R?.4, U5.18 (PGND), U5.19 (PGND)
- new net INOKB: D2.1 (K), Q2.1 (G), U5.2 (INOKB)
- new net ITOPOFF: Q1.2 (D), R17.1, U5.11 (ITOPOFF)
- new net MCU_TEMPSENS: Q1.1 (G), Q2.2 (D), R13.2, R15.2, R16.1
- new net MODE: U4.4 (MODE)
- new net P0_00: U3.F11 (P0-00/XL1)
- new net P0_01: U3.F12 (P0-01/XL2)
- new net P0_02: U3.G11 (P0-02/NFC1)
- new net P0_03: U3.H12 (P0-03/NFC2)
- new net P0_04: U3.G10 (P0-04/AIN0)
- new net P0_05: U3.F10 (P0-05/AIN1)
- new net P0_06: U3.H10 (P0-06/AIN2)
- new net P0_07: U3.J10 (P0-07/AIN3)
- new net P0_08: U3.L12 (P0-08/TRACEDATA3/SCK)
- new net P0_09: U3.J9 (P0-09/TRACEDATA2/MOSI)
- new net P0_10: U3.J8 (P0-10/TRACEDATA1/MISO)
- new net P0_11: U3.J7 (P0-11/TRACEDATA0/~{CS})
- new net P0_12: U3.J6 (P0-12/TRACECLK/DCX)
- new net P0_13: U3.K10 (P0-13/IO0)
- new net P0_14: U3.K9 (P0-14/IO1)
- new net P0_15: U3.L9 (P0-15/IO2)
- new net P0_16: U3.K8 (P0-16/IO3)
- new net P0_17: U3.L7 (P0-17/SCK)
- new net P0_18: U3.K7 (P0-18/~{CS})
- new net P0_19: U3.J5 (P0-19)
- new net P0_20: U3.K5 (P0-20)
- new net P0_21: U3.J4 (P0-21)
- new net P0_22: U3.K4 (P0-22)
- new net P0_23: U3.H3 (P0-23)
- new net P0_24: U3.K2 (P0-24)
- new net P0_25: U3.L1 (P0-25/AIN4)
- new net P0_26: U3.J2 (P0-26/AIN5)
- new net P0_27: U3.H1 (P0-27/AIN6)
- new net P0_28: U3.E3 (P0-28/AIN7)
- new net P0_29: U3.E2 (P0-29)
- new net P0_30: U3.C4 (P0-30)
- new net P0_31: U3.C5 (P0-31)
- new net P1_00: U3.D10 (P1-00)
- new net P1_01: U3.E10 (P1-01)
- new net P1_02: U3.J11 (P1-02/TWI)
- new net P1_03: U3.K12 (P1-03/TWI)
- new net P1_04: U3.K3 (P1-04)
- new net P1_05: U3.L3 (P1-05)
- new net P1_06: U3.J3 (P1-06)
- new net P1_07: U3.G3 (P1-07)
- new net P1_08: U3.F3 (P1-08)
- new net P1_09: U3.H2 (P1-09)
- new net P1_10: U3.E4 (P1-10)
- new net P1_11: U3.C6 (P1-11)
- new net P1_12: U3.C7 (P1-12)
- new net P1_13: U3.C8 (P1-13)
- new net P1_14: U3.C9 (P1-14)
- new net P1_15: U3.C10 (P1-15)
- new net RF_LINE: C35.1, C42.1, L6.2
- new net RX_EN: U4.7 (RX_EN)
- new net SWDCLK: U3.F2 (SWDCLK)
- new net SWDIO: U3.F1 (SWDIO)
- new net TX_EN: U4.9 (TX_EN)
- new net USB_+: J2.A6 (D+), J2.B6 (D+), R5.1, TIE1.2, TIE?.2
- new net USB_-: J2.A7 (D-), J2.B7 (D-), R4.1, TIE1.1, TIE?.1
- new net USB_CC1: J2.A5 (CC1), U5.5 (CC1)
- new net USB_CC2: J2.B5 (CC2), U5.4 (CC2)
- new net VBUS: C9.1, J2.A4 (VBUS), J2.A9 (VBUS), J2.B4 (VBUS), J2.B9 (VBUS), R1.1, U5.23 (CHGIN), U5.24 (CHGIN)
- new net VDD: C17.1, C18.1, C3.1, C4.1, C5.1, C6.1, C7.1, C8.1, U3.A3 (VDD), U3.D2 (VDD), U3.H11 (VDD), U3.K1 (VDD), U3.L11 (VDD), U3.L5 (VDD), U4.5 (VDD), U4.6 (VDD)
- new net owo: R?.3
- new net uwu: R?.2
- new net ~{RESET}: U3.G2 (~{RESET})
- no-connect marks 0 -> 4
Other:
- removed sheet Battery Management
- removed sheet USB & USB PD
- removed sheet nRF52840 Pinout & Supports
- note added: "0"
- note added: "DATE"
- note added: "DESCRIPION OF CHANGE"
- note added: "Fuel Gauge"
- note added: "I don't know what the hell I was doing earlier, but I've realigned, and placed chips where they should be. Finishing up schematic."
- note added: "INOKB control"
- note added: "MAX17262"
- note added: "REV"
- note added: "REVISION HISTORY"
- note added: "Temperature Detection"

Commit message: 
Parts:
- removed AE1, AE2: Antenna, symbol Device:Antenna
- removed BT1: Batt, Connector_JST:JST_EH_S2B-EH_1x02_P2.50mm_Horizontal, symbol Device:Battery_Cell
- removed C16: 10${uF}, Capacitor_Tantalum_SMD:CP_EIA-2012-15_AVX-P, symbol Device:C_Polarized_US
- removed C17, C18, C26, C27, C28, C7, C8: 100nF, Capacitor_SMD:C_0201_0603Metric, symbol Device:C
- removed C19: 1${uF}, Capacitor_SMD:C_0201_0603Metric, symbol Device:C
- removed C20, C23: 1${uF}, Capacitor_SMD:C_0603_1608Metric, symbol Device:C
- removed C21, C22: 2.2nF, Capacitor_SMD:C_0201_0603Metric, symbol Device:C
- removed C24, C25: 4.7${uF}, Capacitor_SMD:C_0805_2012Metric, symbol Device:C
- removed C29: 10${uF}, Capacitor_SMD:C_0805_2012Metric, symbol Device:C
- removed C30, C36: 1.2pF, Capacitor_SMD:C_0201_0603Metric, symbol Device:C
- removed C31, C35, C37: DNP, Capacitor_SMD:C_0201_0603Metric, symbol Device:C
- removed C32, C38: 1.8pF, Capacitor_SMD:C_0201_0603Metric, symbol Device:C
- removed C33, C39: 9.5pF, Capacitor_SMD:C_0201_0603Metric, symbol Device:C
- removed C34: 0.7pF, Capacitor_SMD:C_0201_0603Metric, symbol Device:C
- removed C40, C41: C, Capacitor_SMD:C_0402_1005Metric, symbol Device:C
- removed C42: 1pF, Capacitor_SMD:C_0201_0603Metric, symbol Device:C
- removed C?: 10pF, symbol Device:C
- removed D2: LED_Filled, LED_SMD:LED_0805_2012Metric, symbol Device:LED_Filled
- removed J2: USB_C_Receptacle_USB2.0, Connector_USB:USB_C_Receptacle_Palconn_UTC16-G, symbol Connector:USB_C_Receptacle_USB2.0
- removed L5, L8: NC, Inductor_SMD:L_0402_1005Metric, symbol Device:L
- removed L6: 2.2nH, Inductor_SMD:L_0402_1005Metric, symbol Device:L
- removed L7: 1.9nH, Inductor_SMD:L_0402_1005Metric, symbol Device:L
- removed Q1, Q2: ?, Package_TO_SOT_SMD:SOT-23-5, symbol 4ms_Transistor:PMOS_IRF5305PBF
- removed R10: 470${R}, Resistor_SMD:R_0603_1608Metric, symbol Device:R
- removed R11, R13, R15: 100${kR}, Resistor_SMD:R_0603_1608Metric, symbol Device:R
- removed R12, R14, R18: R, Resistor_SMD:R_0603_1608Metric, symbol Device:R
- removed R16: 1M${R}, Resistor_SMD:R_0603_1608Metric, symbol Device:R
- removed R17: RITOPOFF, Resistor_SMD:R_0603_1608Metric, symbol Device:R
- removed R5: 28${R}, Resistor_SMD:R_0402_1005Metric, symbol Device:R
- removed R6: 0${R}, Resistor_SMD:R_0603_1608Metric, symbol Device:R
- removed R7: 49.9${R}, Resistor_SMD:R_0402_1005Metric, symbol Device:R
- removed R8: CONFIG, Resistor_SMD:R_0603_1608Metric, symbol Device:R
- removed R?: R_Shunt, Resistor_SMD:R_Shunt_Ohmite_LVK12, symbol Device:R_Shunt
- removed R?: 1M${R, symbol Device:R
- removed TH1: Thermistor, Resistor_SMD:R_0603_1608Metric, symbol Device:Thermistor
- removed TIE?: NetTie, 4ms_SolderJumper:Net_Tie_0.16mm_6mil, symbol 4ms_Net-tie:NetTie
- removed U2, U6: MAX9027EBT+T, 0:MAX9027EBT-T, symbol 0.Project:MAX9027EBT+T
- removed U3: NRF5340-CLAA-R, 1.Embedded.Specialized:NRF5340-CLAA-R, symbol 1.Embedded.Specialized:NRF5340-CLAA-R
- removed U4: NRF21540-QDAA-R, Package_DFN_QFN:QFN-16-1EP_3x3mm_P0.5mm_EP1.75x1.75mm, symbol 1.Communications.Amplifiers:NRF21540-QDAA-R
- removed U5: MAX77751CEFG+, 1.Power.BattMgmt:MAX77751CEFG+, symbol 0.Project:MAX77751CEFG+
- removed Y1: 32MHz-ECS-320-8-37B2-7KM-TR, 1.Logic.Oscillators:32MHz-ECS-320-8-37B2-7KM-TR, symbol 1.Logic.Oscillators_Resonators:32MHz-ECS-320-8-37B2-7KM-TR
- added AE1: Antenna_Chip, 0:RF-ANT_A1001312, symbol Device:Antenna_Chip
- added C1: 2.2${uF}, Capacitor_SMD:C_0603_1608Metric, symbol Device:C
- added C2: 10${uF}, Capacitor_SMD:C_0603_1608Metric, symbol Device:C_Polarized_US
- added C? (x2): C, symbol Device:C
- added C? (x15): 100nF, Capacitor_SMD:C_0201_0603Metric, symbol Device:C
- added C?: C, Capacitor_SMD:C_0402_1005Metric, symbol Device:C
- added C? (x3): 1uF, Capacitor_SMD:C_0402_1005Metric, symbol Device:C
- added C?: DNP, Capacitor_SMD:C_0201_0603Metric, symbol Device:C
- added C? (x2): 2.2nF, Capacitor_SMD:C_0201_0603Metric, symbol Device:C
- added C? (x2): 4.7${uF}, Capacitor_SMD:C_0402_1005Metric, symbol Device:C
- added C? (x2): C, Capacitor_SMD:C_0201_0603Metric, symbol Device:C
- added C?: 0.7pF, Capacitor_SMD:C_0201_0603Metric, symbol Device:C
- added D1, D2, D4, D5: LEDAPG0603ZGC-5MAV, LED_SMD:LED_0201_0603Metric, symbol 0.Project:LEDAPG0603ZGC-5MAV
- added D?: LED_Filled, LED_SMD:LED_0402_1005Metric, symbol Device:LED_Filled
- added FB? (x2): FerriteBead, Resistor_SMD:R_0603_1608Metric, symbol Device:FerriteBead
- added H2: H1, MountingHole:MountingHole_2.5mm_Pad, symbol Mechanical:MountingHole_Pad
- added H3: H3, MountingHole:MountingHole_2.5mm_Pad, symbol Mechanical:MountingHole_Pad
- added H4: H4, MountingHole:MountingHole_2.5mm_Pad, symbol Mechanical:MountingHole_Pad
- added J1: Conn_Coaxial, Connector_Coaxial:U.FL_Hirose_U.FL-R-SMT-1_Vertical, symbol Connector:Conn_Coaxial
- added J5: Conn_01x03, 0:JST_ACH_BM03B-ACHSS-GAN-ETF, symbol 4ms_Connector:Conn_01x03
- added J?: USB_C_Receptacle_USB2.0, Connector_USB:USB_C_Receptacle_Palconn_UTC16-G, symbol Connector:USB_C_Receptacle_USB2.0
- added J?: Left Mezzanine, 0:DF40C-80DS-0-4V-51, symbol Connector_Generic:Conn_02x30_Odd_Even
- added L? (x2): 10uH, Inductor_SMD:L_0603_1608Metric, symbol Device:L
- added L?: 2.2nH, Inductor_SMD:L_0402_1005Metric, symbol Device:L
- added Q? (x2): NTND31015NZTAG, 0:NTND31015NZTAG, symbol Device:Q_Dual_PMOS_S1G1D2S2G2D1
- added R19: DNP, Resistor_SMD:R_0402_1005Metric, symbol Device:R
- added R20, R21, R22, R23, R24: R, Resistor_SMD:R_0402_1005Metric, symbol Device:R
- added R37, R38, R39, R40, R41, R9: CONFIG, Resistor_SMD:R_0201_0603Metric, symbol Device:R
- added R8: PCS2512DR0500ET, 0:PCS2512DR0500ET, symbol 0.Project:PCS2512DR0500ET
- added R?: RITOPOFF, Resistor_SMD:R_0201_0603Metric, symbol Device:R
- added R? (x2): 28${R}, Resistor_SMD:R_0201_0603Metric, symbol Device:R
- added R? (x7): R, symbol Device:R
- added R?: 1M${R}, Resistor_SMD:R_0201_0603Metric, symbol Device:R
- added R? (x3): R, Resistor_SMD:R_0201_0603Metric, symbol Device:R
- added R?: 2.2${R}, Resistor_SMD:R_0402_1005Metric, symbol Device:R
- added R? (x3): 100${kR}, Resistor_SMD:R_0201_0603Metric, symbol Device:R
- added R?: 470${R}, Resistor_SMD:R_0201_0603Metric, symbol Device:R
- added TIE?: NetTie, 4ms_SolderJumper:Net_Tie_0.16mm_6mil, symbol 4ms_Net-tie:NetTie
- added TP1, TP2: TestPoint, symbol 4ms_Connector:TestPoint
- added U1: LTC2942, 0:LTC2942, symbol 0.Project:LTC2942
- added U2: MAX77751CEFG+, 1.Power.BattMgmt:MAX77751CEFG+, symbol 0.Project:MAX77751CEFG+
- added U3: NRF21540-QDAA-R, Package_DFN_QFN:QFN-16-1EP_4x4mm_P0.65mm_EP2.1x2.1mm, symbol 1.Communications.Amplifiers:NRF21540-QDAA-R
- added U? (x4): NRF5340-QKAA-R7, 0:NRF5340-QKAA-R7, symbol 1.Embedded.Specialized:NRF5340-QKAA-R7
- added U? (x2): MAX9027EBT+T, 0:MAX9027EBT-T, symbol 0.Project:MAX9027EBT+T
- added U? (x2): PCAL6524, 0:PCAL6524HEHP, symbol 0.Project:PCAL6524
- added U?: W25Q32JVZP, 0:W25QJVZP, symbol 0.Project:W25Q32JVZP
- added Y?: 32MHz-ECS-320-8-37B2-7KM-TR, 1.Logic.Oscillators_Resonators:32MHz-ECS-320-8-37B2-7KM-TR, symbol 1.Logic.Oscillators_Resonators:32MHz-ECS-320-8-37B2-7KM-TR
- added Y?: 32.768kHz, symbol Device:Crystal
- C10: footprint Capacitor_Tantalum_SMD:CP_EIA-2012-15_AVX-P -> Capacitor_SMD:C_0402_1005Metric
- C11: footprint Capacitor_Tantalum_SMD:CP_EIA-2012-15_AVX-P -> Capacitor_SMD:C_0603_1608Metric
- C12: value 100nF -> 2.2${uF}; footprint Capacitor_SMD:C_0201_0603Metric -> Capacitor_SMD:C_0402_1005Metric
- C13: value 2.2${uF} -> 10${uF}; footprint Capacitor_SMD:C_0201_0603Metric -> Capacitor_SMD:C_0603_1608Metric
- C14: footprint Capacitor_SMD:C_0201_0603Metric -> Capacitor_SMD:C_0603_1608Metric
- C15: value 10${uF} -> 1pF
- C4: value 100nF -> 10${uF}; footprint Capacitor_SMD:C_0201_0603Metric -> Capacitor_SMD:C_0603_1608Metric
- C5, C6: value 100nF -> 1.2pF
- C9: value 2.2${uF} -> 100nF; footprint Capacitor_SMD:C_0603_1608Metric -> Capacitor_SMD:C_0201_0603Metric
- L1: value 10${uh} -> 1.9nH; footprint 1.Inductors.L_SRN_LAB2:L_SRN_2016_2010-1R0M -> Inductor_SMD:L_0402_1005Metric
- L3: value 10${uh} -> 4.7nH; footprint 1.Inductors.L_SRN_LAB2:L_SRN_2016_2010-1R0M -> Inductor_SMD:L_0402_1005Metric
- R1: value 2.2${R} -> 0${R}; footprint Resistor_SMD:R_0603_1608Metric -> Resistor_SMD:R_0402_1005Metric
- R2: value 0${R} -> R; footprint Resistor_SMD:R_0603_1608Metric -> Resistor_SMD:R_0402_1005Metric
- R3: value 49.9${R} -> R; Status DNP -> (none)
- R4: value 28${R} -> R
- TIE1: value NetTie -> FL; footprint 4ms_SolderJumper:Net_Tie_0.16mm_6mil -> 0:NetTie_RF_FL
Connections:
- net +5V: now also R?.1, R?.1, R?.1, U?.A1 (V+), U?.A1 (V+); no longer C14.1, C15.1, L2.2
- net +BATT: now also C2.1, R8.1, TP1.1, U1.1 (SENSE+), U2.13 (BATT), U2.14 (BATT)
- net ANT_SEL: now also U3.8 (ANT_SEL)
- net CHARGE_STAT: now also U2.3 (STAT)
- net GNDPWR: now also C12.2, J5.3 (Pin_3), U2.18 (PGND), U2.19 (PGND); no longer C15.2
- net INOKB: now also D?.1 (K), Q?.5 (G), U2.2 (INOKB)
- net ITOPOFF: now also Q?.6 (D), R?.1, U2.11 (ITOPOFF)
- net MCU_TEMPSENS: now also Q?.2 (G), Q?.3 (D), R?.1, R?.2, R?.2
- net MODE: now also U3.4 (MODE)
- net RF_LINE: now also C15.1, C?.1, L?.2
- net RX_EN: now also U3.7 (RX_EN)
- net TX_EN: now also U3.9 (TX_EN)
- net USB_+: now also J?.A6 (D+), J?.B6 (D+), TIE?.2; no longer TIE1.2
- net USB_-: now also J?.A7 (D-), J?.B7 (D-), TIE?.1; no longer R4.1, TIE1.1
- net USB_CC1: now also J?.A5 (CC1), U2.5 (CC1)
- net USB_CC2: now also J?.B5 (CC2), U2.4 (CC2)
- net VBUS: now also C1.1, J?.A4 (VBUS), J?.A9 (VBUS), J?.B4 (VBUS), J?.B9 (VBUS), R?.2, U2.23 (CHGIN), U2.24 (CHGIN); no longer C9.1, R1.1
- net VDD: now also C?.1, C?.1, C?.1, C?.1, C?.1, C?.1, C?.1, C?.1, C?.1, C?.1, C?.1, C?.1, C?.1, R?.2, R?.2, R?.2, R?.2, U2.10 (VDD), U3.5 (VDD), U3.6 (VDD), U?.27 (VDD_{POWER}), U?.31 (VDD_{I2C}), U?.AC1 (VDD), U?.AG1 (VDD), U?.AJ31 (VDD), U?.AL11 (VDD), U?.AL17 (VDD), U?.AL25 (VDD), U?.AL3 (VDD), U?.AL7 (VDD), U?.B28 (VDD), U?.C1 (VDD), U?.E31 (VDD), U?.N31 (VDD), U?.U1 (VDD); no longer C5.1, C6.1
- net +5VP: now reaches C13.1
- net +5VP: now also C14.1, L2.2, U2.15 (SYS), U2.16 (SYS)
- net GND: now reaches R2.2
- net GND: now also C3.2, C4.2, C5.1, C6.1, L3.2, R2.1, R3.1, R3.2, R4.1, R4.2, TIE1.2, AE1.1 (FEED), C1.2, C2.2, C?.2, C?.2, C?.2, C?.2, C?.2, C?.2, C?.2, C?.2, C?.2, C?.2, C?.2, C?.2, C?.2, C?.2, C?.2, C?.2, C?.2, C?.2, C?.2, C?.2, C?.2, C?.2, C?.2, C?.2, C?.2, C?.2, C?.2, C?.2, C?.2, FB?.2, FB?.2, H2.1, H3.1, H4.1, J1.2 (Ext), J?.A1 (GND), J?.A12 (GND), J?.B1 (GND), J?.B12 (GND), Q?.1 (S), Q?.4 (S), R19.2, R20.1, R20.2, R21.1, R21.2, R22.1, R22.2, R23.1, R23.2, R24.1, R24.2, R37.2, R38.2, R39.2, R40.2, R41.2, R9.2, R?.2, R?.2, R?.2, U1.2 (GND), U2.9 (GND), U3.1 (VSS), U3.16 (VSS), U3.17 (VSS), U?.104 (VSS), U?.25 (VSS), U?.35 (VSS), U?.36 (VSS), U?.37 (VSS), U?.38 (VSS), U?.39 (VSS), U?.4 (GND), U?.40 (VSS), U?.41 (VSS), U?.43 (VSS), U?.44 (VSS), U?.45 (VSS), U?.46 (VSS), U?.47 (VSS), U?.48 (VSS), U?.49 (VSS), U?.50 (VSS), U?.51 (VSS), U?.9 (EP), U?.A25 (VSS), U?.A3 (V-), U?.A3 (V-), U?.B12 (VSS), U?.B2 (V-), U?.B2 (V-), U?.B26 (VSS), U?.EPAD (VSS), U?.G1 (VSS), U?.H2 (VSS), U?.J31 (VSS), Y?.2, Y?.4
- net at L2.1: now also C9.2, U2.20 (LX), U2.21 (LX); no longer C12.2
- net at L3.1: now also C5.2, L1.2, R1.1, R19.1
- net ANT2_OUT: now reaches L1.1
- net ANT2_OUT: now also U3.3 (ANT2)
- net at R1.2: now also TIE1.1, AE1.2 (PCB_Trace)
- net PWR_VBYP: now reaches C10.1, C11.1
- net PWR_VBYP: now also U2.22 (BYP)
- net ANT1_OUT: now reaches L4.1
- net ANT1_OUT: now also U3.2 (ANT1)
- net at C12.1: now also U2.17 (PVL)
- removed net AVSS: C3.2, C4.2, C5.2, C6.2, C9.2, R3.2
- new net: C6.2, J1.1 (In), L4.2
- new net: R?.1, R?.2
- new net: R?.2, R?.2
- new net: C9.1, U2.1 (BST)
- new net: D4.1 (K), R39.1
- new net: C?.1, R?.1, Y?.1
- new net: D?.2 (A), R?.2
- new net: C?.1, U?.B30 (XC2), Y?.1
- new net: C?.1, U?.C31 (XC1), Y?.3
- new net: R9.1, U2.12 (IFAST)
- new net: C15.2, U3.10 (TRX)
- new net: D1.1 (K), R37.1
- new net: R?.1, R?.2, U?.B3 (-)
- new net: C?.1, U?.A13 (DECA)
- new net: J5.1 (Pin_1), R8.2, TP2.1, U1.6 (SENSE-)
- new net: C?.1, R?.1, U?.A5 (VBUS)
- new net: C?.1, R?.1, Y?.2
- new net: FB?.1, FB?.1, J?.S1 (SHIELD)
- new net: C?.1, L?.1 (x2)
- new net: D5.1 (K), R40.1
- new net: C?.1, U?.A23 (DECN)
- new net: R?.1, U?.A2 (x2)
- new net: R?.1, R?.2, U?.B1 (+)
- new net: U?.A1 (NC), U?.A31 (NC), U?.AG31 (NC), U?.AL1 (NC), U?.AL31 (NC), U?.D2 (NC), U?.F2 (NC), U?.K2 (NC), U?.T2 (NC)
- new net: D2.1 (K), R38.1
- new net: C?.1, U?.B6 (DECUSB)
- new net: C?.1, L?.1, U?.L31 (ANT)
- new net ${SHEETNAME}_P0_0: U?.1 (P0_0)
- new net ${SHEETNAME}_P0_1: U?.2 (P0_1)
- new net ${SHEETNAME}_P0_2: U?.3 (P0_2)
- new net ${SHEETNAME}_P0_3: U?.4 (P0_3)
- new net ${SHEETNAME}_P0_4: U?.5 (P0_4)
- new net ${SHEETNAME}_P0_5: U?.6 (P0_5)
- new net ${SHEETNAME}_P0_6: U?.7 (P0_6)
- new net ${SHEETNAME}_P0_7: U?.8 (P0_7)
- new net ${SHEETNAME}_P1_0: U?.9 (P1_0)
- new net ${SHEETNAME}_P1_1: U?.10 (P1_1)
- new net ${SHEETNAME}_P1_2: U?.11 (P1_2)
- new net ${SHEETNAME}_P1_3: U?.12 (P1_3)
- new net ${SHEETNAME}_P1_4: U?.13 (P1_4)
- new net ${SHEETNAME}_P1_5: U?.14 (P1_5)
- new net ${SHEETNAME}_P1_6: U?.15 (P1_6)
- new net ${SHEETNAME}_P1_7: U?.16 (P1_7)
- new net ${SHEETNAME}_P2_0: U?.17 (P2_0)
- new net ${SHEETNAME}_P2_1: U?.18 (P2_1)
- new net ${SHEETNAME}_P2_2: U?.19 (P2_2)
- new net ${SHEETNAME}_P2_3: U?.20 (P2_3)
- new net ${SHEETNAME}_P2_4: U?.21 (P2_4)
- new net ${SHEETNAME}_P2_5: U?.22 (P2_5)
- new net ${SHEETNAME}_P2_6: U?.23 (P2_6)
- new net ${SHEETNAME}_P2_7: U?.24 (P2_7)
- new net ${SHEETNAME}_~{INT}: R?.1, U?.32 (~{INT})
- new net ${SHEETNAME}_~{RESET}: R?.1, U?.28 (~{RESET})
- new net +3V3: C?.1, U?.8 (VCC)
- new net ADDR: U?.26 (ADDR)
- new net BATT_ALARM: U1.5 (~{AL}/CC)
- new net BATT_I2C_SCL: U1.3 (SCL)
- new net BATT_I2C_SDA: U1.4 (SDA)
- new net ENBST_CTRL: R41.1, U2.8 (ENBST)
- new net NRF.P0_00: U?.N1 (P0.00/XL1)
- new net NRF.P0_01: U?.R1 (P0.01/XL2)
- new net NRF.P0_02: U?.W1 (P0.02/NFC1)
- new net NRF.P0_03: U?.AA1 (P0.03/NFC2)
- new net NRF.P0_04: U?.V2 (P0.04/AIN0)
- new net NRF.P0_05: U?.Y2 (P0.05/AIN1)
- new net NRF.P0_06: U?.AB2 (P0.06/AIN2)
- new net NRF.P0_07: U?.AD2 (P0.07/AIN3)
- new net NRF.P0_08: U?.AH2 (P0.08/TRACEDATA[3]/SCK)
- new net NRF.P0_09: U?.AJ1 (P0.09/TRACEDATA[2]/MOSI)
- new net NRF.P0_10: U?.AK2 (P0.10/TRACEDATA[1]/MISO)
- new net NRF.P0_11: U?.AK4 (P0.11/TRACEDATA[0]/CSN)
- new net NRF.P0_12: U?.AK6 (P0.12/TRACECLK/DCX)
- new net NRF.P0_19: U?.AL13 (P0.19)
- new net NRF.P0_20: U?.AK16 (P0.20)
- new net NRF.P0_21: U?.AL15 (P0.21)
- new net NRF.P0_22: U?.AK18 (P0.22)
- new net NRF.P0_23: U?.AK20 (P0.23)
- new net NRF.P0_24: U?.AL27 (P0.24)
- new net NRF.P0_25: U?.AK28 (P0.25/AIN4)
- new net NRF.P0_26: U?.AL29 (P0.26/AIN5)
- new net NRF.P0_27: U?.AK30 (P0.27/AIN6)
- new net NRF.P0_28: U?.AE31 (P0.28/AIN7)
- new net NRF.P0_29: U?.U31 (P0.29)
- new net NRF.P0_30: U?.B24 (P0.30)
- new net NRF.P0_31: U?.B22 (P0.31)
- new net NRF.P1_00: U?.M2 (P1.00)
- new net NRF.P1_01: U?.P2 (P1.01)
- new net NRF.P1_02: U?.AE1 (P1.02/TWI)
- new net NRF.P1_03: U?.AF2 (P1.03/TWI)
- new net NRF.P1_04: U?.AL19 (P1.04)
- new net NRF.P1_05: U?.AK22 (P1.05)
- new net NRF.P1_06: U?.AL21 (P1.06)
- new net NRF.P1_07: U?.AK24 (P1.07)
- new net NRF.P1_08: U?.AL23 (P1.08)
- new net NRF.P1_09: U?.AK26 (P1.09)
- new net NRF.P1_10: U?.R31 (P1.10)
- new net NRF.P1_11: U?.B20 (P1.11)
- new net NRF.P1_12: U?.B18 (P1.12)
- new net NRF.P1_13: U?.A17 (P1.13)
- new net NRF.P1_14: U?.B16 (P1.14)
- new net NRF.P1_15: U?.B14 (P1.15)
- new net NRF_IFX.SWDCLK: U?.W31 (SWDCLK)
- new net NRF_IFX.SWDIO: U?.AA31 (SWDIO)
- new net NRF_IFX.USB_+: R?.1
- new net NRF_IFX.USB_-: R?.1
- new net NRF_IFX.~{RESET}: U?.AC31 (~{RESET})
- new net QSPI_IO_0: U?.5 (DI(IO0)), U?.AL5 (P0.13/IO[0])
- new net QSPI_IO_1: U?.2 (DO(IO1)), U?.AK8 (P0.14/IO[1])
- new net QSPI_IO_2: U?.3 (IO2), U?.AK10 (P0.15/IO[2])
- new net QSPI_IO_3: U?.7 (IO3), U?.AL9 (P0.16/IO[3])
- new net QSPI_SCK: U?.6 (CLK), U?.AK12 (P0.17/SCK)
- new net QSPI_~{CS}: U?.1 (~{CS}), U?.AK14 (P0.18/CSN)
- new net SCL: R?.1, U?.29 (SCL)
- new net SDA: R?.1, U?.30 (SDA)
- new net nrf_D+: R?.2, U?.B2 (D+)
- new net nrf_D-: R?.2, U?.B4 (D-)
- new net therm: J5.2 (Pin_2), R?.2, U?.B1 (+), U?.B3 (-)
Other:
- note added: "MAX77751 * ENBST, IFAST, INOKB, STAT indication, jumpers, switches * Exact components recommended by https://www.analog.com/media/en/technical-documentation/data-sheets/MAX77751CEVKIT-MAX77751FEVKIT.pdf * Output to buck/boost/ldo regulator for 5V + 3.3V rails Buck-Boost * High efficiency, <$5 buck-boost IC for high loads LDO * Replace buck-boost if possible."
- note added: "Place Near Antenna"
- note removed: "Fuel Gauge"
- note removed: "MAX17262"

Commit message: 
Parts:
- removed AE1: Antenna_Chip, 0:RF-ANT_A1001312, symbol Device:Antenna_Chip
- removed C1: 2.2${uF}, Capacitor_SMD:C_0603_1608Metric, symbol Device:C
- removed C10: 10${uF}, Capacitor_SMD:C_0402_1005Metric, symbol Device:C_Polarized_US
- removed C11: 22${uF}, Capacitor_SMD:C_0603_1608Metric, symbol Device:C_Polarized_US
- removed C12: 2.2${uF}, Capacitor_SMD:C_0402_1005Metric, symbol Device:C
- removed C13, C14, C4: 10${uF}, Capacitor_SMD:C_0603_1608Metric, symbol Device:C
- removed C15: 1pF, Capacitor_SMD:C_0201_0603Metric, symbol Device:C
- removed C2: 10${uF}, Capacitor_SMD:C_0603_1608Metric, symbol Device:C_Polarized_US
- removed C3, C9, C? (x15): 100nF, Capacitor_SMD:C_0201_0603Metric, symbol Device:C
- removed C5, C6: 1.2pF, Capacitor_SMD:C_0201_0603Metric, symbol Device:C
- removed C? (x2): C, symbol Device:C
- removed C?: C, Capacitor_SMD:C_0402_1005Metric, symbol Device:C
- removed C? (x3): 1uF, Capacitor_SMD:C_0402_1005Metric, symbol Device:C
- removed C?: DNP, Capacitor_SMD:C_0201_0603Metric, symbol Device:C
- removed C? (x2): 2.2nF, Capacitor_SMD:C_0201_0603Metric, symbol Device:C
- removed C? (x2): 4.7${uF}, Capacitor_SMD:C_0402_1005Metric, symbol Device:C
- removed C? (x2): C, Capacitor_SMD:C_0201_0603Metric, symbol Device:C
- removed C?: 0.7pF, Capacitor_SMD:C_0201_0603Metric, symbol Device:C
- removed D1, D2, D4, D5: LEDAPG0603ZGC-5MAV, LED_SMD:LED_0201_0603Metric, symbol 0.Project:LEDAPG0603ZGC-5MAV
- removed D?: LED_Filled, LED_SMD:LED_0402_1005Metric, symbol Device:LED_Filled
- removed FB? (x2): FerriteBead, Resistor_SMD:R_0603_1608Metric, symbol Device:FerriteBead
- removed H2: H1, MountingHole:MountingHole_2.5mm_Pad, symbol Mechanical:MountingHole_Pad
- removed H3: H3, MountingHole:MountingHole_2.5mm_Pad, symbol Mechanical:MountingHole_Pad
- removed H4: H4, MountingHole:MountingHole_2.5mm_Pad, symbol Mechanical:MountingHole_Pad
- removed J1: Conn_Coaxial, Connector_Coaxial:U.FL_Hirose_U.FL-R-SMT-1_Vertical, symbol Connector:Conn_Coaxial
- removed J5: Conn_01x03, 0:JST_ACH_BM03B-ACHSS-GAN-ETF, symbol 4ms_Connector:Conn_01x03
- removed J?: USB_C_Receptacle_USB2.0, Connector_USB:USB_C_Receptacle_Palconn_UTC16-G, symbol Connector:USB_C_Receptacle_USB2.0
- removed J?: Left Mezzanine, 0:DF40C-80DS-0-4V-51, symbol Connector_Generic:Conn_02x30_Odd_Even
- removed L1, L4: 1.9nH, Inductor_SMD:L_0402_1005Metric, symbol Device:L
- removed L2: 0.47${uh}, 1.Inductors.L_SRN_LAB2:L_SRN_2016_2012-R47M, symbol 1.Inductors.L_SRN_LAB2:L_SRN_2016_2010-R47M
- removed L3: 4.7nH, Inductor_SMD:L_0402_1005Metric, symbol Device:L
- removed L? (x2): 10uH, Inductor_SMD:L_0603_1608Metric, symbol Device:L
- removed L?: 2.2nH, Inductor_SMD:L_0402_1005Metric, symbol Device:L
- removed Q? (x2): NTND31015NZTAG, 0:NTND31015NZTAG, symbol Device:Q_Dual_PMOS_S1G1D2S2G2D1
- removed R1: 0${R}, Resistor_SMD:R_0402_1005Metric, symbol Device:R
- removed R19: DNP, Resistor_SMD:R_0402_1005Metric, symbol Device:R
- removed R2, R20, R21, R22, R23, R24, R3, R4: R, Resistor_SMD:R_0402_1005Metric, symbol Device:R
- removed R37, R38, R39, R40, R41, R9: CONFIG, Resistor_SMD:R_0201_0603Metric, symbol Device:R
- removed R8: PCS2512DR0500ET, 0:PCS2512DR0500ET, symbol 0.Project:PCS2512DR0500ET
- removed R?: RITOPOFF, Resistor_SMD:R_0201_0603Metric, symbol Device:R
- removed R? (x2): 28${R}, Resistor_SMD:R_0201_0603Metric, symbol Device:R
- removed R? (x7): R, symbol Device:R
- removed R?: 1M${R}, Resistor_SMD:R_0201_0603Metric, symbol Device:R
- removed R? (x3): R, Resistor_SMD:R_0201_0603Metric, symbol Device:R
- removed R?: 2.2${R}, Resistor_SMD:R_0402_1005Metric, symbol Device:R
- removed R? (x3): 100${kR}, Resistor_SMD:R_0201_0603Metric, symbol Device:R
- removed R?: 470${R}, Resistor_SMD:R_0201_0603Metric, symbol Device:R
- removed TIE1: FL, 0:NetTie_RF_FL, symbol 4ms_Net-tie:NetTie
- removed TIE?: NetTie, 4ms_SolderJumper:Net_Tie_0.16mm_6mil, symbol 4ms_Net-tie:NetTie
- removed TP1, TP2: TestPoint, symbol 4ms_Connector:TestPoint
- removed U1: LTC2942, 0:LTC2942, symbol 0.Project:LTC2942
- removed U2: MAX77751CEFG+, 1.Power.BattMgmt:MAX77751CEFG+, symbol 0.Project:MAX77751CEFG+
- removed U3: NRF21540-QDAA-R, Package_DFN_QFN:QFN-16-1EP_4x4mm_P0.65mm_EP2.1x2.1mm, symbol 1.Communications.Amplifiers:NRF21540-QDAA-R
- removed U? (x4): NRF5340-QKAA-R7, 0:NRF5340-QKAA-R7, symbol 1.Embedded.Specialized:NRF5340-QKAA-R7
- removed U? (x2): MAX9027EBT+T, 0:MAX9027EBT-T, symbol 0.Project:MAX9027EBT+T
- removed U? (x2): PCAL6524, 0:PCAL6524HEHP, symbol 0.Project:PCAL6524
- removed U?: W25Q32JVZP, 0:W25QJVZP, symbol 0.Project:W25Q32JVZP
- removed Y?: 32MHz-ECS-320-8-37B2-7KM-TR, 1.Logic.Oscillators_Resonators:32MHz-ECS-320-8-37B2-7KM-TR, symbol 1.Logic.Oscillators_Resonators:32MHz-ECS-320-8-37B2-7KM-TR
- removed Y?: 32.768kHz, symbol Device:Crystal
Connections:
- no-connect marks 4 -> 0
Other:
- added sheet Battery Management (schematics/battery_mgmt/battery_mgmt.kicad_sch)
- added sheet IO Expansion (schematics/io_expansion/io_expansion.kicad_sch)
- added sheet Mechanical (schematics/mechanical/mechanical.kicad_sch)
- added sheet Microcontroller (schematics/mcu/mcu.kicad_sch)
- added sheet Power (schematics/power/power.kicad_sch)
- added sheet RF Section (schematics/rf/rf.kicad_sch)
- added sheet USB Interface (schematics/usb/usb.kicad_sch)
- note removed: "0"
- note removed: "DATE"
- note removed: "DESCRIPION OF CHANGE"
- note removed: "I don't know what the hell I was doing earlier, but I've realigned, and placed chips where they should be. Finishing up schematic."
- note removed: "INOKB control"
- note removed: "MAX77751 * ENBST, IFAST, INOKB, STAT indication, jumpers, switches * Exact components recommended by https://www.analog.com/media/en/technical-documentation/data-sheets/MAX77751CEVKIT-MAX77751FEVKIT.pdf * Output to buck/boost/ldo regulator for 5V + 3.3V rails Buck-Boost * High efficiency, <$5 buck-boost IC for high loads LDO * Replace buck-boost if possible."
- note removed: "Place Near Antenna"
- note removed: "REV"
- note removed: "REVISION HISTORY"
- note removed: "Temperature Detection"
