File: hw/schematics/rf/rf.kicad_sch (KiCad schematic)
At the start: 22 parts, among them J1 Conn_Coaxial, U3 NRF21540-QDAA-R

Commit message: 
Other:
- moved on the sheet: AE1, C15, C3, C4, C5, C6, J1, L1, L3, L4, R1, R19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
